File: hardware/mcu.kicad_sch (KiCad schematic)
At the start: 21 parts, among them J1 UART MCU, SW1 BOOT, SW2 RESET, U15 VEML7700, U3 ESP32-WROVER-E

Commit message: Assign footprints
Parts:
- BZ1: footprint (none) -> Transducer_espena:TP094003_Transducer_9x9mm
- C12, C5: footprint (none) -> Capacitor_SMD:C_0805_2012Metric
- J1: footprint (none) -> Connector_espena:Magnetic-Pogo-Female-MG0425FB_1x4_P2.54mm
- R12, R13, R14, R15, R16, R17, R18, R19, R2: footprint (none) -> Resistor_SMD:R_0805_2012Metric
- SW1, SW2: footprint (none) -> Button_Switch_SMD_espena:SW_SPST_TL3301_6x6mm_H4.3mm
Changed lines of the file:
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@@
       (effects (font (size 0.762 0.762)) (justify left))
     )
-    (property "Footprint" "" (at 90.17 81.28 0)
+    (property "Footprint" "Capacitor_SMD:C_0805_2012Metric" (at 90.17 81.28 0)
       (effects (font (size 1.27 1.27)) hide)
     )
@@
       (effects (font (size 1.27 1.27)) (justify right))
     )
-    (property "Footprint" "" (at 191.262 38.1 90)
+    (property "Footprint" "Resistor_SMD:R_0805_2012Metric" (at 191.262 38.1 90)
       (effects (font (size 1.27 1.27)) hide)
     )
@@
       (effects (font (size 1.27 1.27)) (justify right))
     )
-    (property "Footprint" "" (at 191.262 124.46 90)
+    (property "Footprint" "Resistor_SMD:R_0805_2012Metric" (at 191.262 124.46 90)
       (effects (font (size 1.27 1.27)) hide)
     )
@@
       (effects (font (size 1.27 1.27)) (justify right))
     )
-    (property "Footprint" "" (at 83.312 34.29 90)
+    (property "Footprint" "Resistor_SMD:R_0805_2012Metric" (at 83.312 34.29 90)
       (effects (font (size 1.27 1.27)) hide)
     )
@@
       (effects (font (size 1.27 1.27)) (justify right))
     )
-    (property "Footprint" "" (at 89.408 72.39 90)
+    (property "Footprint" "Resistor_SMD:R_0805_2012Metric" (at 89.408 72.39 90)
       (effects (font (size 1.27 1.27)) hide)
     )
@@
       (effects (font (size 1.27 1.27)) (justify right))
     )
-    (property "Footprint" "" (at 154.432 154.305 90)
+    (property "Footprint" "Resistor_SMD:R_0805_2012Metric" (at 154.432 154.305 90)
       (effects (font (size 1.27 1.27)) hide)
     )
@@
       (effects (font (size 1.27 1.27)) (justify right))
     )
-    (property "Footprint" "" (at 191.262 63.5 90)
+    (property "Footprint" "Resistor_SMD:R_0805_2012Metric" (at 191.262 63.5 90)
       (effects (font (size 1.27 1.27)) hide)
     )
@@
       (effects (font (size 1.27 1.27)))
     )
-    (property "Footprint" "" (at 123.19 40.64 0)
+    (property "Footprint" "Button_Switch_SMD_espena:SW_SPST_TL3301_6x6mm_H4.3mm" (at 123.19 40.64 0)
       (effects (font (size 1.27 1.27)) hide)
     )
@@
       (effects (font (size 1.27 1.27)))
     )
-    (property "Footprint" "" (at 106.68 116.84 0)
+    (property "Footprint" "Connector_espena:Magnetic-Pogo-Female-MG0425FB_1x4_P2.54mm" (at 106.68 116.84 0)
       (effects (font (size 1.27 1.27)) hide)
     )
@@
       (effects (font (size 1.27 1.27)) (justify right))
     )
-    (property "Footprint" "" (at 191.262 134.62 90)
+    (property "Footprint" "Resistor_SMD:R_0805_2012Metric" (at 191.262 134.62 90)
       (effects (font (size 1.27 1.27)) hide)
     )
@@
       (effects (font (size 1.27 1.27)))
     )
-    (property "Footprint" "" (at 123.19 135.89 0)
+    (property "Footprint" "Button_Switch_SMD_espena:SW_SPST_TL3301_6x6mm_H4.3mm" (at 123.19 135.89 0)
       (effects (font (size 1.27 1.27)) hide)
     )
@@
       (effects (font (size 1.27 1.27)) (justify left))
     )
-    (property "Footprint" "" (at 135.255 53.34 90)
+    (property "Footprint" "Transducer_espena:TP094003_Transducer_9x9mm" (at 135.255 53.34 90)
       (effects (font (size 1.27 1.27)) hide)
     )
@@
       (effects (font (size 1.27 1.27)) (justify right))
     )
-    (property "Footprint" "" (at 92.202 34.29 90)
+    (property "Footprint" "Resistor_SMD:R_0805_2012Metric" (at 92.202 34.29 90)
       (effects (font (size 1.27 1.27)) hide)
     )
@@
       (effects (font (size 0.762 0.762)) (justify left))
     )
-    (property "Footprint" "" (at 157.48 33.02 0)
+    (property "Footprint" "Capacitor_SMD:C_0805_2012Metric" (at 157.48 33.02 0)
       (effects (font (size 1.27 1.27)) hide)
     )
@@
       (effects (font (size 1.27 1.27)) (justify right))
     )
-    (property "Footprint" "" (at 132.842 35.56 90)
+    (property "Footprint" "Resistor_SMD:R_0805_2012Metric" (at 132.842 35.56 90)
       (effects (font (size 1.27 1.27)) hide)
     )
@@
       (effects (font (size 1.27 1.27)) (justify right))
     )
-    (property "Footprint" "" (at 132.842 133.35 90)
+    (property "Footprint" "Resistor_SMD:R_0805_2012Metric" (at 132.842 133.35 90)
       (effects (font (size 1.27 1.27)) hide)
     )
@@
       (effects (font (size 1.27 1.27)) (justify right))
     )
-    (property "Footprint" "" (at 135.5852 151.13 0)
+    (property "Footprint" "Capacitor_SMD:C_0805_2012Metric" (at 135.5852 151.13 0)
       (effects (font (size 1.27 1.27)) hide)
     )
@@
       (effects (font (size 0.762 0.762)) (justify left))
     )
-    (property "Footprint" "" (at 85.09 81.28 0)
+    (property "Footprint" "Capacitor_SMD:C_0805_2012Metric" (at 85.09 81.28 0)
       (effects (font (size 1.27 1.27)) hide)
     )
@@
       (effects (font (size 1.27 1.27)) (justify right))
     )
-    (property "Footprint" "" (at 136.398 110.49 90)
-      (effects (font (size 1.27 1.27)) hide)
-    )
+    (property "Footprint" "Resistor_SMD:R_0805_2012Metric" (at 136.398 110.49 90)
+      (effects (font (size 1.27 1.27)) hide)
+    )
