File: hardware/mcu.kicad_sch (KiCad schematic)
At the start: 20 parts, among them J1 UART MCU, SW1 BOOT, SW2 RESET, U15 VEML7700, U3 ESP32-WROVER-E

Commit message: Updated project to work with KiCAD version 9
Parts:
- U3: footprint RF_Module_espena:ESP32-WROVER-B -> RF_Module_espena:ESP32-WROVER-E
