File: hardware/mcu_2.kicad_sch (KiCad schematic)
At the start: 20 parts, among them J1 UART MCU, SW1 BOOT, SW2 RESET, U15 VEML7700, U3 ESP32-WROVER-E

Commit message: Starting PCB routing process
Parts:
- removed BZ1: Buzzer, Transducer_espena:TP094003_Transducer_9x9mm, symbol Device_espena:Buzzer
- removed C12: 1uF, Capacitor_SMD:C_0805_2012Metric, symbol Device:C
- removed C13: 47uF, Capacitor_SMD:C_0805_2012Metric, symbol Device_espena:C_Decoupling
- removed C22: 100nF, Capacitor_SMD:C_0805_2012Metric, symbol Device_espena:C_Decoupling
- removed C23: 10μF, Capacitor_SMD:C_0805_2012Metric, symbol Device_espena:C_Decoupling
- removed J1: UART MCU, Connector_espena:Magnetic-Pogo-Female-MG0425FB_1x4_P2.54mm, symbol Connector_Generic:Conn_01x04
- removed R12: 4,7k, Resistor_SMD:R_0805_2012Metric, symbol Device:R
- removed R13, R2: 4.7k, Resistor_SMD:R_0805_2012Metric, symbol Device:R
- removed R14, R15, R16, R22: 10k, Resistor_SMD:R_0805_2012Metric, symbol Device:R
- removed R17, R18, R19: 4k7, Resistor_SMD:R_0805_2012Metric, symbol Device:R
- removed SW1: BOOT, Button_Switch_SMD_espena:SW_SPST_TL3301_6x6mm_H4.3mm, symbol Switch:SW_Push
- removed SW2: RESET, Button_Switch_SMD_espena:SW_SPST_TL3301_6x6mm_H4.3mm, symbol Switch:SW_Push
- removed U15: VEML7700, Sensor_espena:VEML7700, symbol Sensor_Optical_espena:VEML7700
- removed U3: ESP32-WROVER-E, RF_Module_espena:ESP32-WROVER-B, symbol RF_Module_espena:ESP32-WROVER-E
- added BZ2: Buzzer, Transducer_espena:TP094003_Transducer_9x9mm, symbol Device_espena:Buzzer
- added C25: 10μF, Capacitor_SMD:C_0805_2012Metric, symbol Device_espena:C_Decoupling
- added C29: 100nF, Capacitor_SMD:C_0805_2012Metric, symbol Device_espena:C_Decoupling
- added C30: 1uF, Capacitor_SMD:C_0805_2012Metric, symbol Device:C
- added C33: 47uF, Capacitor_SMD:C_0805_2012Metric, symbol Device_espena:C_Decoupling
- added J4: UART MCU, Connector_espena:Magnetic-Pogo-Female-MG0425FB_1x4_P2.54mm, symbol Connector_Generic:Conn_01x04
- added R23, R25, R27, R28: 4k7, Resistor_SMD:R_0805_2012Metric, symbol Device:R
- added R26: 4.7k, Resistor_SMD:R_0805_2012Metric, symbol Device:R
- added R29, R31, R32, R33: 10k, Resistor_SMD:R_0805_2012Metric, symbol Device:R
- added R30: 4.7k, symbol Device:R
- added SW3: BOOT, Button_Switch_SMD_espena:SW_SPST_TL3301_6x6mm_H4.3mm, symbol Switch:SW_Push
- added SW4: RESET, Button_Switch_SMD_espena:SW_SPST_TL3301_6x6mm_H4.3mm, symbol Switch:SW_Push
- added U16: VEML7700, symbol Sensor_Optical_espena:VEML7700
- added U17: ESP32-WROVER-E, RF_Module_espena:ESP32-WROVER-E, symbol RF_Module_espena:ESP32-WROVER-E
Connections:
- net DIAL_BLANK: now also U17.30 (IO18)
- net DIAL_DCPRG: now also U17.37 (IO23)
- net DIAL_GSCLK: now also U17.12 (IO27)
- net DIAL_SCLK: now also U17.11 (IO26)
- net DIAL_SIN: now also U17.9 (IO33)
- net DIAL_SOUT: now also U17.8 (IO32)
- net DIAL_VPRG: now also U17.31 (IO19)
- net DIAL_XERR: now also U17.5 (I39)
- net DIAL_XLAT: now also U17.10 (IO25)
- net DISP_SPI_CLK: now also U17.13 (IO14)
- net DISP_SPI_MISO: now also R31.1, U17.14 (IO12)
- net DISP_SPI_MOSI: now also U17.16 (IO13)
- net DISP_U1BLINK: now also U17.7 (I35)
- net DISP_U2BLINK: now also U17.4 (I36)
- net GND: now also BZ2.2 (+), C25.2, C29.2, C30.2, C33.2, J4.4 (Pin_4), R29.2, R31.2, R33.2, SW3.1, SW4.1, U16. (V_{DD}), U17.1 (GND1), U17.15 (GND2), U17.38 (GND3)
- net GPS_TIMEPULSE: now also R32.1, R33.1, U17.6 (I34)
- net SCL: now also R25.2, U16. (V_{DD}), U17.36 (IO22)
- net SDA: now also R23.2, U16. (V_{DD}), U17.33 (IO21)
- net ~{DISP_SPI_CS}: now also R30.2, U17.23 (IO15)
- new net: C33.1, U17.2 (3V3)
- new net: R29.1, U17.24 (IO2)
- new net: R26.2, SW3.2, U17.25 (IO0)
- new net: BZ2.1 (-), U17.29 (IO5)
- new net: C30.1, R28.2, SW4.2, U17.3 (EN)
- new net: J4.3 (Pin_3), U17.34 (RXD0)
- new net: J4.2 (Pin_2), R27.2, U17.35 (TXD0)
- new net: C25.1, C29.1
