File: hardware/broadcast_clock.kicad_pcb (KiCad board)
At the start: 2 copper layers, 239.5 x 239.5 mm, 354 parts

Commit message: Starting PCB routing process
Parts:
- added AE1: Active GPS antenna 3.3V, Connector_Coaxial:SMA_Amphenol_132291-12_Vertical, B.Cu at (40.4, 45.1)
- added BT1: CR 2032, Battery:BatteryHolder_Keystone_1058_1x2032, B.Cu at (49.8, 64.8)
- added BZ1: Buzzer, Transducer_espena:TP094003_Transducer_9x9mm, B.Cu at (255.4, 39.9)
- added C1: 26pF, Capacitor_SMD:C_0805_2012Metric, F.Cu at (68.2, 150.5)
- added C10: 100nF, Capacitor_SMD:C_0805_2012Metric, F.Cu at (107.1, 90.4)
- added C11: 100nF, Capacitor_SMD:C_0805_2012Metric, F.Cu at (138.7, 230.4)
- added C12: 1uF, Capacitor_SMD:C_0805_2012Metric, B.Cu at (250.3, 35.2)
- added C13: 47uF, Capacitor_SMD:C_0805_2012Metric, B.Cu at (245.9, 35.2)
- added C14: 820uF, Capacitor_SMD_espena:CP_Elec_18x16.5, B.Cu at (38.4, 211.1)
- added C15: 100uF, Capacitor_SMD:CP_Elec_8x10, B.Cu at (59.7, 230.9)
- added C16: 40nF, Capacitor_SMD:C_0805_2012Metric, B.Cu at (70.1, 240.5)
- added C17: 10nF, Capacitor_SMD:C_0805_2012Metric, B.Cu at (48.0, 40.0)
- added C18: 47pF, Capacitor_SMD:C_0805_2012Metric, B.Cu at (48.1, 47.6)
- added C19: 820uF, Capacitor_SMD_espena:CP_Elec_18x16.5, B.Cu at (38.1, 87.9)
- added C2: 100nF, Capacitor_SMD:C_0805_2012Metric, F.Cu at (68.2, 142.0)
- added C20: 100nF, Capacitor_SMD:C_0805_2012Metric, B.Cu at (42.7, 191.8)
- added C21: 10µF, Capacitor_SMD:C_0805_2012Metric, B.Cu at (35.9, 194.3)
- added C22: 100nF, Capacitor_SMD:C_0805_2012Metric, F.Cu at (151.0, 117.4)
- added C23: 10μF, Capacitor_SMD:C_0805_2012Metric, F.Cu at (139.8, 117.4)
- added C24: 10µF, Capacitor_SMD:C_0805_2012Metric, B.Cu at (103.6, 183.5)
- added C26: 100nF, Capacitor_SMD:C_0805_2012Metric, B.Cu at (40.6, 38.6)
- added C27: 10µF, Capacitor_SMD:C_0805_2012Metric, B.Cu at (218.4, 116.6)
- added C28: 820uF, Capacitor_SMD_espena:CP_Elec_18x16.5, B.Cu at (88.4, 38.1)
- added C3: 100nF, Capacitor_SMD:C_0805_2012Metric, F.Cu at (238.1, 140.9)
- added C31: 100nF, Capacitor_SMD:C_0805_2012Metric, B.Cu at (222.2, 116.6)
- added C32: 100nF, Capacitor_SMD:C_0805_2012Metric, B.Cu at (107.4, 183.5)
- added C4: 26pF, Capacitor_SMD:C_0805_2012Metric, F.Cu at (238.4, 150.7)
- added C5: 47uF, Capacitor_SMD:C_0805_2012Metric, F.Cu at (70.4, 142.0)
- added C6: 47uF, Capacitor_SMD:C_0805_2012Metric, F.Cu at (240.4, 140.9)
- added C7: 100nF, Capacitor_SMD:C_0805_2012Metric, F.Cu at (197.1, 90.4)
- added C8: 100nF, Capacitor_SMD:C_0805_2012Metric, F.Cu at (183.8, 200.4)
- added C9: 100nF, Capacitor_SMD:C_0805_2012Metric, F.Cu at (93.9, 200.4)
- added D355: SK33, Diode_SMD:D_SMA, B.Cu at (62.5, 240.5)
- added D356: CMS04, Diode_SMD_mouser:SODFL4724X108N, B.Cu at (40.6, 231.4)
- added D357: 470nm, LED_SMD:LED_0805_2012Metric, F.Cu at (115.3, 29.4)
- added D358: 570nm, LED_SMD:LED_0805_2012Metric, F.Cu at (135.4, 29.4)
- added D359: 590nm, LED_SMD:LED_0805_2012Metric, F.Cu at (155.4, 29.4)
- added D360: 620nm, LED_SMD:LED_0805_2012Metric, F.Cu at (175.5, 29.4)
- added F1: 2A, Fuse_espena:FuseHolder_Keystone_3554, B.Cu at (32.8, 228.3)
- added J1: UART MCU, Connector_espena:Magnetic-Pogo-Female-MG0425FB_1x4_P2.54mm, B.Cu at (215.5, 44.6)
- added J2: POWER, Connector_BarrelJack_espena:BarrelJack_DC044_Horizontal, B.Cu at (48.5, 230.3)
- added J3: UART GPS, Connector_PinHeader_1.27mm:PinHeader_1x06_P1.27mm_Vertical, B.Cu at (73.2, 32.6)
- added L1: 37uH, Inductor_SMD_espena:L_Pulse_LCI-44, B.Cu at (84.3, 252.7)
- added L2: 27nH, Inductor_SMD_espena:L_Coilcraft_0805CS, B.Cu at (48.1, 45.1)
- added R1: 53.6k, Resistor_SMD:R_0805_2012Metric, F.Cu at (52.7, 150.7)
- added R10: 2k, Resistor_SMD:R_0805_2012Metric, F.Cu at (140.9, 225.3)
- added R11: R, Resistor_SMD:R_0805_2012Metric, F.Cu at (240.4, 37.7)
- added R12: 4,7k, Resistor_SMD:R_0805_2012Metric, B.Cu at (245.9, 38.9)
- added R13: 4.7k, Resistor_SMD:R_0805_2012Metric, B.Cu at (222.0, 46.2)
- added R14: 10k, Resistor_SMD:R_0805_2012Metric, B.Cu at (245.9, 49.9)
- added R15: 10k, Resistor_SMD:R_0805_2012Metric, B.Cu at (245.9, 53.6)
- added R16: 10k, Resistor_SMD:R_0805_2012Metric, B.Cu at (222.0, 49.9)
- added R17: 4k7, Resistor_SMD:R_0805_2012Metric, B.Cu at (222.0, 35.2)
- added R18: 4k7, Resistor_SMD:R_0805_2012Metric, B.Cu at (222.0, 42.5)
- added R19: 4k7, Resistor_SMD:R_0805_2012Metric, B.Cu at (222.0, 38.9)
- added R2: 4.7k, Resistor_SMD:R_0805_2012Metric, B.Cu at (222.0, 53.6)
- added R20: 5.6kΩ, Resistor_SMD:R_0805_2012Metric, B.Cu at (72.6, 240.5)
- added R21: 1kΩ, Resistor_SMD:R_0805_2012Metric, B.Cu at (67.6, 240.5)
- added R213: 10k, Resistor_SMD:R_0805_2012Metric, F.Cu at (227.4, 44.7)
- added R22: 10k, Resistor_SMD:R_0805_2012Metric, B.Cu at (245.9, 42.6)
- added R24: 10Ω, Resistor_SMD:R_0805_2012Metric, B.Cu at (48.1, 42.6)
- added R3: 4.7k, Resistor_SMD:R_0805_2012Metric, F.Cu at (222.9, 155.7)
- added R4: R, Resistor_SMD:R_0805_2012Metric, F.Cu at (52.7, 156.1)
- added R5: 53.6k, Resistor_SMD:R_0805_2012Metric, F.Cu at (222.9, 150.5)
- added R6: 2k, Resistor_SMD:R_0805_2012Metric, F.Cu at (194.9, 95.6)
- added R7: 2k, Resistor_SMD:R_0805_2012Metric, F.Cu at (185.9, 195.3)
- added R8: 2k, Resistor_SMD:R_0805_2012Metric, F.Cu at (96.0, 195.3)
- added R9: 2k, Resistor_SMD:R_0805_2012Metric, F.Cu at (104.7, 95.7)
- added SW1: BOOT, Button_Switch_SMD_espena:SW_SPST_TL3301_6x6mm_H4.3mm, B.Cu at (254.3, 59.9)
- added SW2: RESET, Button_Switch_SMD_espena:SW_SPST_TL3301_6x6mm_H4.3mm, B.Cu at (254.3, 69.7)
- added U1: MAX6952, Package_SO_espena:SSOP-36_7.5x12.5mm_P0.65mm, F.Cu at (60.4, 145.4)
- added U10: NCP1117-5.0, Package_TO_SOT_SMD:SOT-223-3_TabPin2, B.Cu at (37.2, 188.7)
- added U11: LM2596DS-ADJ, Regulator_SMD_mouser:NCP5663DSADJR4G, B.Cu at (66.8, 258.5)
- added U12: NCP1117-3.3, Package_TO_SOT_SMD:SOT-223-3_TabPin2, B.Cu at (39.6, 33.0)
- added U13: NCP1117-3.3, Package_TO_SOT_SMD:SOT-223-3_TabPin2, B.Cu at (105.5, 177.3)
- added U14: NCP1117-3.3, Package_TO_SOT_SMD:SOT-223-3_TabPin2, B.Cu at (220.4, 110.4)
- added U15: VEML7700, Sensor_espena:VEML7700, F.Cu at (145.4, 117.1)
- added U2: MAX6952, Package_SO_espena:SSOP-36_7.5x12.5mm_P0.65mm, F.Cu at (230.4, 145.4)
- added U3: ESP32-WROVER-E, RF_Module_espena:ESP32-WROVER-B, B.Cu at (242.8, 33.6)
- added U4: TLC5940PWP, Package_SO_espena:HTSSOP-28-1EP_4.4x9.7mm_P0.65mm_EP3.4x9.5mm_Mask2.4x6.17mm_ThermalVias, F.Cu at (190.4, 90.4)
- added U5: TLC5940PWP, Package_SO_espena:HTSSOP-28-1EP_4.4x9.7mm_P0.65mm_EP3.4x9.5mm_Mask2.4x6.17mm_ThermalVias, B.Cu at (190.4, 200.4)
- added U6: TLC5940PWP, Package_SO_espena:HTSSOP-28-1EP_4.4x9.7mm_P0.65mm_EP3.4x9.5mm_Mask2.4x6.17mm_ThermalVias, B.Cu at (100.4, 200.4)
- added U7: TLC5940PWP, Package_SO_espena:HTSSOP-28-1EP_4.4x9.7mm_P0.65mm_EP3.4x9.5mm_Mask2.4x6.17mm_ThermalVias, B.Cu at (100.4, 90.4)
- added U8: TLC5940PWP, Package_SO_espena:HTSSOP-28-1EP_4.4x9.7mm_P0.65mm_EP3.4x9.5mm_Mask2.4x6.17mm_ThermalVias, B.Cu at (145.4, 230.4)
- added U9: LEA-M8T, RF_GPS_espena:ublox_LEA, B.Cu at (59.9, 40.4)
- D1, D10, D100, D101, D102, D103, D104, D105, D106, D107, D108, D109, D11, D110, D111, D112, D113, D114, D115, D116, D117, D118, D119, D12, D120, D121, D122, D123, D124, D125, D126, D127, D128, D129, D13, D130, D131, D132, D133, D134, D135, D136, D137, D138, D139, D14, D140, D141, D142, D143, D144, D145, D146, D147, D148, D149, D15, D150, D151, D152, D153, D154, D155, D156, D157, D158, D159, D16, D160, D161, D162, D163, D164, D165, D166, D167, D168, D169, D17, D170, D171, D172, D173, D174, D175, D176, D177, D178, D179, D18, D180, D181, D182, D183, D184, D185, D186, D187, D188, D189, D19, D190, D191, D192, D193, D194, D195, D196, D197, D198, D199, D2, D20, D200, D201, D202, D203, D204, D205, D206, D207, D208, D209, D21, D210, D211, D212, D213, D214, D215, D216, D217, D218, D219, D22, D220, D221, D222, D223, D224, D225, D226, D227, D228, D229, D23, D230, D231, D232, D233, D234, D235, D236, D237, D238, D239, D24, D240, D241, D242, D243, D244, D245, D246, D247, D248, D249, D25, D250, D251, D252, D253, D254, D255, D256, D257, D258, D259, D26, D260, D261, D262, D263, D264, D265, D266, D267, D268, D269, D27, D270, D271, D272, D273, D274, D275, D276, D277, D278, D279, D28, D280, D281, D282, D283, D284, D285, D286, D287, D288, D289, D29, D290, D291, D292, D293, D294, D295, D296, D297, D298, D299, D3, D30, D300, D301, D302, D303, D304, D305, D306, D307, D308, D309, D31, D310, D311, D312, D313, D314, D315, D316, D317, D318, D319, D32, D320, D321, D322, D323, D324, D325, D326, D327, D328, D329, D33, D330, D331, D332, D333, D334, D335, D336, D337, D338, D339, D34, D340, D341, D342, D343, D344, D345, D346, D347, D348, D349, D35, D350, D351, D352, D353, D354, D36, D37, D38, D39, D4, D40, D41, D42, D43, D44, D45, D46, D47, D48, D49, D5, D50, D51, D52, D53, D54, D55, D56, D57, D58, D59, D6, D60, D61, D62, D63, D64, D65, D66, D67, D68, D69, D7, D70, D71, D72, D73, D74, D75, D76, D77, D78, D79, D8, D80, D81, D82, D83, D84, D85, D86, D87, D88, D89, D9, D90, D91, D92, D93, D94, D95, D96, D97, D98, D99: value (none) -> 620nm
Connections:
- D1 pad 1: (no net) -> Net-(D1-K)
- D1 pad 2: (no net) -> Net-(D1-A)
- D10 pad 1: (no net) -> Net-(D10-K)
- D10 pad 2: (no net) -> Net-(D1-A)
- D100 pad 1: (no net) -> /Clock face/LED display/LED matrices/U1D0D1R7
- D100 pad 2: (no net) -> /Clock face/LED display/LED matrices/U1D0D2C4
- D101 pad 1: (no net) -> /Clock face/LED display/LED matrices/U1D0D1R1
- D101 pad 2: (no net) -> /Clock face/LED display/LED matrices/U1D0D2C5
- D102 pad 1: (no net) -> /Clock face/LED display/LED matrices/U1D0D1R2
- D102 pad 2: (no net) -> /Clock face/LED display/LED matrices/U1D0D2C5
- D103 pad 1: (no net) -> /Clock face/LED display/LED matrices/U1D0D1R3
- D103 pad 2: (no net) -> /Clock face/LED display/LED matrices/U1D0D2C5
- D104 pad 1: (no net) -> /Clock face/LED display/LED matrices/U1D0D1R4
- D104 pad 2: (no net) -> /Clock face/LED display/LED matrices/U1D0D2C5
- D105 pad 1: (no net) -> /Clock face/LED display/LED matrices/U1D0D1R5
- D105 pad 2: (no net) -> /Clock face/LED display/LED matrices/U1D0D2C5
- D106 pad 1: (no net) -> /Clock face/LED display/LED matrices/U1D0D1R6
- D106 pad 2: (no net) -> /Clock face/LED display/LED matrices/U1D0D2C5
- D107 pad 1: (no net) -> /Clock face/LED display/LED matrices/U1D0D1R7
- D107 pad 2: (no net) -> /Clock face/LED display/LED matrices/U1D0D2C5
- D108 pad 1: (no net) -> /Clock face/LED display/LED matrices/U1D0D1R1
- D108 pad 2: (no net) -> /Clock face/LED display/LED matrices/U1D1D3C1
- D109 pad 1: (no net) -> /Clock face/LED display/LED matrices/U1D0D1R2
- D109 pad 2: (no net) -> /Clock face/LED display/LED matrices/U1D1D3C1
- D11 pad 1: (no net) -> Net-(D11-K)
- D11 pad 2: (no net) -> Net-(D1-A)
- D110 pad 1: (no net) -> /Clock face/LED display/LED matrices/U1D0D1R3
- D110 pad 2: (no net) -> /Clock face/LED display/LED matrices/U1D1D3C1
- D111 pad 1: (no net) -> /Clock face/LED display/LED matrices/U1D0D1R4
- D111 pad 2: (no net) -> /Clock face/LED display/LED matrices/U1D1D3C1
- D112 pad 1: (no net) -> /Clock face/LED display/LED matrices/U1D0D1R5
- D112 pad 2: (no net) -> /Clock face/LED display/LED matrices/U1D1D3C1
- D113 pad 1: (no net) -> /Clock face/LED display/LED matrices/U1D0D1R6
- D113 pad 2: (no net) -> /Clock face/LED display/LED matrices/U1D1D3C1
- D114 pad 1: (no net) -> /Clock face/LED display/LED matrices/U1D0D1R7
- D114 pad 2: (no net) -> /Clock face/LED display/LED matrices/U1D1D3C1
- D115 pad 1: (no net) -> /Clock face/LED display/LED matrices/U1D0D1R1
- D115 pad 2: (no net) -> /Clock face/LED display/LED matrices/U1D1D3C2
- D116 pad 1: (no net) -> /Clock face/LED display/LED matrices/U1D0D1R2
- D116 pad 2: (no net) -> /Clock face/LED display/LED matrices/U1D1D3C2
- D117 pad 1: (no net) -> /Clock face/LED display/LED matrices/U1D0D1R3
- D117 pad 2: (no net) -> /Clock face/LED display/LED matrices/U1D1D3C2
- D118 pad 1: (no net) -> /Clock face/LED display/LED matrices/U1D0D1R4
- D118 pad 2: (no net) -> /Clock face/LED display/LED matrices/U1D1D3C2
- D119 pad 1: (no net) -> /Clock face/LED display/LED matrices/U1D0D1R5
- D119 pad 2: (no net) -> /Clock face/LED display/LED matrices/U1D1D3C2
- D12 pad 1: (no net) -> Net-(D12-K)
- D12 pad 2: (no net) -> Net-(D1-A)
- D120 pad 1: (no net) -> /Clock face/LED display/LED matrices/U1D0D1R6
- D120 pad 2: (no net) -> /Clock face/LED display/LED matrices/U1D1D3C2
- D121 pad 1: (no net) -> /Clock face/LED display/LED matrices/U1D0D1R7
- D121 pad 2: (no net) -> /Clock face/LED display/LED matrices/U1D1D3C2
- D122 pad 1: (no net) -> /Clock face/LED display/LED matrices/U1D0D1R1
- D122 pad 2: (no net) -> /Clock face/LED display/LED matrices/U1D1D3C3
- D123 pad 1: (no net) -> /Clock face/LED display/LED matrices/U1D0D1R2
- D123 pad 2: (no net) -> /Clock face/LED display/LED matrices/U1D1D3C3
- D124 pad 1: (no net) -> /Clock face/LED display/LED matrices/U1D0D1R3
- D124 pad 2: (no net) -> /Clock face/LED display/LED matrices/U1D1D3C3
- D125 pad 1: (no net) -> /Clock face/LED display/LED matrices/U1D0D1R4
- D125 pad 2: (no net) -> /Clock face/LED display/LED matrices/U1D1D3C3
- D126 pad 1: (no net) -> /Clock face/LED display/LED matrices/U1D0D1R5
- D126 pad 2: (no net) -> /Clock face/LED display/LED matrices/U1D1D3C3
- D127 pad 1: (no net) -> /Clock face/LED display/LED matrices/U1D0D1R6
- D127 pad 2: (no net) -> /Clock face/LED display/LED matrices/U1D1D3C3
- D128 pad 1: (no net) -> /Clock face/LED display/LED matrices/U1D0D1R7
- D128 pad 2: (no net) -> /Clock face/LED display/LED matrices/U1D1D3C3
- D129 pad 1: (no net) -> /Clock face/LED display/LED matrices/U1D0D1R1
- D129 pad 2: (no net) -> /Clock face/LED display/LED matrices/U1D1D3C4
- D13 pad 1: (no net) -> Net-(D13-K)
- D13 pad 2: (no net) -> Net-(D1-A)
- D130 pad 1: (no net) -> /Clock face/LED display/LED matrices/U1D0D1R2
- D130 pad 2: (no net) -> /Clock face/LED display/LED matrices/U1D1D3C4
- D131 pad 1: (no net) -> /Clock face/LED display/LED matrices/U1D0D1R3
- D131 pad 2: (no net) -> /Clock face/LED display/LED matrices/U1D1D3C4
- D132 pad 1: (no net) -> /Clock face/LED display/LED matrices/U1D0D1R4
- D132 pad 2: (no net) -> /Clock face/LED display/LED matrices/U1D1D3C4
- D133 pad 1: (no net) -> /Clock face/LED display/LED matrices/U1D0D1R5
- D133 pad 2: (no net) -> /Clock face/LED display/LED matrices/U1D1D3C4
- D134 pad 1: (no net) -> /Clock face/LED display/LED matrices/U1D0D1R6
- D134 pad 2: (no net) -> /Clock face/LED display/LED matrices/U1D1D3C4
- D135 pad 1: (no net) -> /Clock face/LED display/LED matrices/U1D0D1R7
- D135 pad 2: (no net) -> /Clock face/LED display/LED matrices/U1D1D3C4
- D136 pad 1: (no net) -> /Clock face/LED display/LED matrices/U1D0D1R1
- D136 pad 2: (no net) -> /Clock face/LED display/LED matrices/U1D1D3C5
- D137 pad 1: (no net) -> /Clock face/LED display/LED matrices/U1D0D1R2
- D137 pad 2: (no net) -> /Clock face/LED display/LED matrices/U1D1D3C5
- D138 pad 1: (no net) -> /Clock face/LED display/LED matrices/U1D0D1R3
- D138 pad 2: (no net) -> /Clock face/LED display/LED matrices/U1D1D3C5
- D139 pad 1: (no net) -> /Clock face/LED display/LED matrices/U1D0D1R4
- D139 pad 2: (no net) -> /Clock face/LED display/LED matrices/U1D1D3C5
- D14 pad 1: (no net) -> Net-(D14-K)
- D14 pad 2: (no net) -> Net-(D1-A)
- D140 pad 1: (no net) -> /Clock face/LED display/LED matrices/U1D0D1R5
- D140 pad 2: (no net) -> /Clock face/LED display/LED matrices/U1D1D3C5
- D141 pad 1: (no net) -> /Clock face/LED display/LED matrices/U1D0D1R6
- D141 pad 2: (no net) -> /Clock face/LED display/LED matrices/U1D1D3C5
- D142 pad 1: (no net) -> /Clock face/LED display/LED matrices/U1D0D1R7
- D142 pad 2: (no net) -> /Clock face/LED display/LED matrices/U1D1D3C5
- D143 pad 1: (no net) -> /Clock face/LED display/LED matrices/U1D2D3R1
- D143 pad 2: (no net) -> /Clock face/LED display/LED matrices/U1D0D2C1
- D144 pad 1: (no net) -> /Clock face/LED display/LED matrices/U1D2D3R2
- D144 pad 2: (no net) -> /Clock face/LED display/LED matrices/U1D0D2C1
- D145 pad 1: (no net) -> /Clock face/LED display/LED matrices/U1D2D3R3
- D145 pad 2: (no net) -> /Clock face/LED display/LED matrices/U1D0D2C1
- D146 pad 1: (no net) -> /Clock face/LED display/LED matrices/U1D2D3R4
- D146 pad 2: (no net) -> /Clock face/LED display/LED matrices/U1D0D2C1
- D147 pad 1: (no net) -> /Clock face/LED display/LED matrices/U1D2D3R5
- D147 pad 2: (no net) -> /Clock face/LED display/LED matrices/U1D0D2C1
- D148 pad 1: (no net) -> /Clock face/LED display/LED matrices/U1D2D3R6
- D148 pad 2: (no net) -> /Clock face/LED display/LED matrices/U1D0D2C1
- D149 pad 1: (no net) -> /Clock face/LED display/LED matrices/U1D2D3R7
- D149 pad 2: (no net) -> /Clock face/LED display/LED matrices/U1D0D2C1
- D15 pad 1: (no net) -> Net-(D15-K)
- D15 pad 2: (no net) -> Net-(D1-A)
- D150 pad 1: (no net) -> /Clock face/LED display/LED matrices/U1D2D3R1
- D150 pad 2: (no net) -> /Clock face/LED display/LED matrices/U1D0D2C2
- D151 pad 1: (no net) -> /Clock face/LED display/LED matrices/U1D2D3R2
- D151 pad 2: (no net) -> /Clock face/LED display/LED matrices/U1D0D2C2
- D152 pad 1: (no net) -> /Clock face/LED display/LED matrices/U1D2D3R3
- D152 pad 2: (no net) -> /Clock face/LED display/LED matrices/U1D0D2C2
- D153 pad 1: (no net) -> /Clock face/LED display/LED matrices/U1D2D3R4
- D153 pad 2: (no net) -> /Clock face/LED display/LED matrices/U1D0D2C2
- D154 pad 1: (no net) -> /Clock face/LED display/LED matrices/U1D2D3R5
- D154 pad 2: (no net) -> /Clock face/LED display/LED matrices/U1D0D2C2
- D155 pad 1: (no net) -> /Clock face/LED display/LED matrices/U1D2D3R6
- D155 pad 2: (no net) -> /Clock face/LED display/LED matrices/U1D0D2C2
- D156 pad 1: (no net) -> /Clock face/LED display/LED matrices/U1D2D3R7
- D156 pad 2: (no net) -> /Clock face/LED display/LED matrices/U1D0D2C2
- D157 pad 1: (no net) -> /Clock face/LED display/LED matrices/U1D2D3R1
- D157 pad 2: (no net) -> /Clock face/LED display/LED matrices/U1D0D2C3
- D158 pad 1: (no net) -> /Clock face/LED display/LED matrices/U1D2D3R2
- D158 pad 2: (no net) -> /Clock face/LED display/LED matrices/U1D0D2C3
- D159 pad 1: (no net) -> /Clock face/LED display/LED matrices/U1D2D3R3
- D159 pad 2: (no net) -> /Clock face/LED display/LED matrices/U1D0D2C3
- D16 pad 1: (no net) -> Net-(D16-K)
- D16 pad 2: (no net) -> Net-(D1-A)
- D160 pad 1: (no net) -> /Clock face/LED display/LED matrices/U1D2D3R4
- D160 pad 2: (no net) -> /Clock face/LED display/LED matrices/U1D0D2C3
- D161 pad 1: (no net) -> /Clock face/LED display/LED matrices/U1D2D3R5
- D161 pad 2: (no net) -> /Clock face/LED display/LED matrices/U1D0D2C3
- D162 pad 1: (no net) -> /Clock face/LED display/LED matrices/U1D2D3R6
- D162 pad 2: (no net) -> /Clock face/LED display/LED matrices/U1D0D2C3
- D163 pad 1: (no net) -> /Clock face/LED display/LED matrices/U1D2D3R7
- D163 pad 2: (no net) -> /Clock face/LED display/LED matrices/U1D0D2C3
- D164 pad 1: (no net) -> /Clock face/LED display/LED matrices/U1D2D3R1
- D164 pad 2: (no net) -> /Clock face/LED display/LED matrices/U1D0D2C4
- D165 pad 1: (no net) -> /Clock face/LED display/LED matrices/U1D2D3R2
- D165 pad 2: (no net) -> /Clock face/LED display/LED matrices/U1D0D2C4
- D166 pad 1: (no net) -> /Clock face/LED display/LED matrices/U1D2D3R3
- D166 pad 2: (no net) -> /Clock face/LED display/LED matrices/U1D0D2C4
- D167 pad 1: (no net) -> /Clock face/LED display/LED matrices/U1D2D3R4
- D167 pad 2: (no net) -> /Clock face/LED display/LED matrices/U1D0D2C4
- D168 pad 1: (no net) -> /Clock face/LED display/LED matrices/U1D2D3R5
- D168 pad 2: (no net) -> /Clock face/LED display/LED matrices/U1D0D2C4
- D169 pad 1: (no net) -> /Clock face/LED display/LED matrices/U1D2D3R6
- D169 pad 2: (no net) -> /Clock face/LED display/LED matrices/U1D0D2C4
- D17 pad 1: (no net) -> Net-(D17-K)
- D17 pad 2: (no net) -> Net-(D1-A)
- D170 pad 1: (no net) -> /Clock face/LED display/LED matrices/U1D2D3R7
- D170 pad 2: (no net) -> /Clock face/LED display/LED matrices/U1D0D2C4
- D171 pad 1: (no net) -> /Clock face/LED display/LED matrices/U1D2D3R1
- D171 pad 2: (no net) -> /Clock face/LED display/LED matrices/U1D0D2C5
- D172 pad 1: (no net) -> /Clock face/LED display/LED matrices/U1D2D3R2
- D172 pad 2: (no net) -> /Clock face/LED display/LED matrices/U1D0D2C5
- D173 pad 1: (no net) -> /Clock face/LED display/LED matrices/U1D2D3R3
- D173 pad 2: (no net) -> /Clock face/LED display/LED matrices/U1D0D2C5
- D174 pad 1: (no net) -> /Clock face/LED display/LED matrices/U1D2D3R4
- D174 pad 2: (no net) -> /Clock face/LED display/LED matrices/U1D0D2C5
- D175 pad 1: (no net) -> /Clock face/LED display/LED matrices/U1D2D3R5
- D175 pad 2: (no net) -> /Clock face/LED display/LED matrices/U1D0D2C5
- D176 pad 1: (no net) -> /Clock face/LED display/LED matrices/U1D2D3R6
- D176 pad 2: (no net) -> /Clock face/LED display/LED matrices/U1D0D2C5
- D177 pad 1: (no net) -> /Clock face/LED display/LED matrices/U1D2D3R7
- D177 pad 2: (no net) -> /Clock face/LED display/LED matrices/U1D0D2C5
- D178 pad 1: (no net) -> /Clock face/LED display/LED matrices/U1D2D3R1
- D178 pad 2: (no net) -> /Clock face/LED display/LED matrices/U1D1D3C1
- D179 pad 1: (no net) -> /Clock face/LED display/LED matrices/U1D2D3R2
- D179 pad 2: (no net) -> /Clock face/LED display/LED matrices/U1D1D3C1
- D18 pad 1: (no net) -> Net-(D18-K)
- D18 pad 2: (no net) -> Net-(D1-A)
- D180 pad 1: (no net) -> /Clock face/LED display/LED matrices/U1D2D3R3
- D180 pad 2: (no net) -> /Clock face/LED display/LED matrices/U1D1D3C1
- D181 pad 1: (no net) -> /Clock face/LED display/LED matrices/U1D2D3R4
- D181 pad 2: (no net) -> /Clock face/LED display/LED matrices/U1D1D3C1
- D182 pad 1: (no net) -> /Clock face/LED display/LED matrices/U1D2D3R5
- D182 pad 2: (no net) -> /Clock face/LED display/LED matrices/U1D1D3C1
- D183 pad 1: (no net) -> /Clock face/LED display/LED matrices/U1D2D3R6
- D183 pad 2: (no net) -> /Clock face/LED display/LED matrices/U1D1D3C1
- D184 pad 1: (no net) -> /Clock face/LED display/LED matrices/U1D2D3R7
- D184 pad 2: (no net) -> /Clock face/LED display/LED matrices/U1D1D3C1
- D185 pad 1: (no net) -> /Clock face/LED display/LED matrices/U1D2D3R1
- D185 pad 2: (no net) -> /Clock face/LED display/LED matrices/U1D1D3C2
- D186 pad 1: (no net) -> /Clock face/LED display/LED matrices/U1D2D3R2
- D186 pad 2: (no net) -> /Clock face/LED display/LED matrices/U1D1D3C2
- D187 pad 1: (no net) -> /Clock face/LED display/LED matrices/U1D2D3R3
- D187 pad 2: (no net) -> /Clock face/LED display/LED matrices/U1D1D3C2
- D188 pad 1: (no net) -> /Clock face/LED display/LED matrices/U1D2D3R4
- D188 pad 2: (no net) -> /Clock face/LED display/LED matrices/U1D1D3C2
- D189 pad 1: (no net) -> /Clock face/LED display/LED matrices/U1D2D3R5
- D189 pad 2: (no net) -> /Clock face/LED display/LED matrices/U1D1D3C2
- D19 pad 1: (no net) -> Net-(D19-K)
- D19 pad 2: (no net) -> Net-(D1-A)
- D190 pad 1: (no net) -> /Clock face/LED display/LED matrices/U1D2D3R6
- D190 pad 2: (no net) -> /Clock face/LED display/LED matrices/U1D1D3C2
- D191 pad 1: (no net) -> /Clock face/LED display/LED matrices/U1D2D3R7
- D191 pad 2: (no net) -> /Clock face/LED display/LED matrices/U1D1D3C2
- D192 pad 1: (no net) -> /Clock face/LED display/LED matrices/U1D2D3R1
- D192 pad 2: (no net) -> /Clock face/LED display/LED matrices/U1D1D3C3
- D193 pad 1: (no net) -> /Clock face/LED display/LED matrices/U1D2D3R2
- D193 pad 2: (no net) -> /Clock face/LED display/LED matrices/U1D1D3C3
- D194 pad 1: (no net) -> /Clock face/LED display/LED matrices/U1D2D3R3
- D194 pad 2: (no net) -> /Clock face/LED display/LED matrices/U1D1D3C3
- D195 pad 1: (no net) -> /Clock face/LED display/LED matrices/U1D2D3R4
- D195 pad 2: (no net) -> /Clock face/LED display/LED matrices/U1D1D3C3
- D196 pad 1: (no net) -> /Clock face/LED display/LED matrices/U1D2D3R5
- D196 pad 2: (no net) -> /Clock face/LED display/LED matrices/U1D1D3C3
- D197 pad 1: (no net) -> /Clock face/LED display/LED matrices/U1D2D3R6
- D197 pad 2: (no net) -> /Clock face/LED display/LED matrices/U1D1D3C3
- D198 pad 1: (no net) -> /Clock face/LED display/LED matrices/U1D2D3R7
- D198 pad 2: (no net) -> /Clock face/LED display/LED matrices/U1D1D3C3
- D199 pad 1: (no net) -> /Clock face/LED display/LED matrices/U1D2D3R1
- D199 pad 2: (no net) -> /Clock face/LED display/LED matrices/U1D1D3C4
- D2 pad 1: (no net) -> Net-(D2-K)
- D2 pad 2: (no net) -> Net-(D1-A)
- D20 pad 1: (no net) -> Net-(D20-K)
- D20 pad 2: (no net) -> Net-(D1-A)
- D200 pad 1: (no net) -> /Clock face/LED display/LED matrices/U1D2D3R2
- D200 pad 2: (no net) -> /Clock face/LED display/LED matrices/U1D1D3C4
- D201 pad 1: (no net) -> /Clock face/LED display/LED matrices/U1D2D3R3
- D201 pad 2: (no net) -> /Clock face/LED display/LED matrices/U1D1D3C4
- D202 pad 1: (no net) -> /Clock face/LED display/LED matrices/U1D2D3R4
- D202 pad 2: (no net) -> /Clock face/LED display/LED matrices/U1D1D3C4
- D203 pad 1: (no net) -> /Clock face/LED display/LED matrices/U1D2D3R5
- D203 pad 2: (no net) -> /Clock face/LED display/LED matrices/U1D1D3C4
- D204 pad 1: (no net) -> /Clock face/LED display/LED matrices/U1D2D3R6
- D204 pad 2: (no net) -> /Clock face/LED display/LED matrices/U1D1D3C4
- D205 pad 1: (no net) -> /Clock face/LED display/LED matrices/U1D2D3R7
- D205 pad 2: (no net) -> /Clock face/LED display/LED matrices/U1D1D3C4
- D206 pad 1: (no net) -> /Clock face/LED display/LED matrices/U1D2D3R1
- D206 pad 2: (no net) -> /Clock face/LED display/LED matrices/U1D1D3C5
- D207 pad 1: (no net) -> /Clock face/LED display/LED matrices/U1D2D3R2
- D207 pad 2: (no net) -> /Clock face/LED display/LED matrices/U1D1D3C5
- D208 pad 1: (no net) -> /Clock face/LED display/LED matrices/U1D2D3R3
- D208 pad 2: (no net) -> /Clock face/LED display/LED matrices/U1D1D3C5
- D209 pad 1: (no net) -> /Clock face/LED display/LED matrices/U1D2D3R4
- D209 pad 2: (no net) -> /Clock face/LED display/LED matrices/U1D1D3C5
- D21 pad 1: (no net) -> Net-(D21-K)
- D21 pad 2: (no net) -> Net-(D1-A)
- D210 pad 1: (no net) -> /Clock face/LED display/LED matrices/U1D2D3R5
- D210 pad 2: (no net) -> /Clock face/LED display/LED matrices/U1D1D3C5
- D211 pad 1: (no net) -> /Clock face/LED display/LED matrices/U1D2D3R6
- D211 pad 2: (no net) -> /Clock face/LED display/LED matrices/U1D1D3C5
- D212 pad 1: (no net) -> /Clock face/LED display/LED matrices/U1D2D3R7
- D212 pad 2: (no net) -> /Clock face/LED display/LED matrices/U1D1D3C5
- D213 pad 1: (no net) -> /Clock face/LED display/LED matrices/U2D0D1R1
- D213 pad 2: (no net) -> /Clock face/LED display/LED matrices/U2D0D2C1
- D214 pad 1: (no net) -> /Clock face/LED display/LED matrices/U2D0D1R2
- D214 pad 2: (no net) -> /Clock face/LED display/LED matrices/U2D0D2C1
- D215 pad 1: (no net) -> /Clock face/LED display/LED matrices/U2D0D1R3
- D215 pad 2: (no net) -> /Clock face/LED display/LED matrices/U2D0D2C1
- D216 pad 1: (no net) -> /Clock face/LED display/LED matrices/U2D0D1R4
- D216 pad 2: (no net) -> /Clock face/LED display/LED matrices/U2D0D2C1
- D217 pad 1: (no net) -> /Clock face/LED display/LED matrices/U2D0D1R5
- D217 pad 2: (no net) -> /Clock face/LED display/LED matrices/U2D0D2C1
- D218 pad 1: (no net) -> /Clock face/LED display/LED matrices/U2D0D1R6
- D218 pad 2: (no net) -> /Clock face/LED display/LED matrices/U2D0D2C1
- D219 pad 1: (no net) -> /Clock face/LED display/LED matrices/U2D0D1R7
- D219 pad 2: (no net) -> /Clock face/LED display/LED matrices/U2D0D2C1
- D22 pad 1: (no net) -> Net-(D22-K)
- D22 pad 2: (no net) -> Net-(D1-A)
- D220 pad 1: (no net) -> /Clock face/LED display/LED matrices/U2D0D1R1
- D220 pad 2: (no net) -> /Clock face/LED display/LED matrices/U2D0D2C2
- D221 pad 1: (no net) -> /Clock face/LED display/LED matrices/U2D0D1R2
- D221 pad 2: (no net) -> /Clock face/LED display/LED matrices/U2D0D2C2
- D222 pad 1: (no net) -> /Clock face/LED display/LED matrices/U2D0D1R3
- D222 pad 2: (no net) -> /Clock face/LED display/LED matrices/U2D0D2C2
- D223 pad 1: (no net) -> /Clock face/LED display/LED matrices/U2D0D1R4
- D223 pad 2: (no net) -> /Clock face/LED display/LED matrices/U2D0D2C2
- D224 pad 1: (no net) -> /Clock face/LED display/LED matrices/U2D0D1R5
- D224 pad 2: (no net) -> /Clock face/LED display/LED matrices/U2D0D2C2
- D225 pad 1: (no net) -> /Clock face/LED display/LED matrices/U2D0D1R6
- D225 pad 2: (no net) -> /Clock face/LED display/LED matrices/U2D0D2C2
- D226 pad 1: (no net) -> /Clock face/LED display/LED matrices/U2D0D1R7
- D226 pad 2: (no net) -> /Clock face/LED display/LED matrices/U2D0D2C2
- D227 pad 1: (no net) -> /Clock face/LED display/LED matrices/U2D0D1R1
- D227 pad 2: (no net) -> /Clock face/LED display/LED matrices/U2D0D2C3
- D228 pad 1: (no net) -> /Clock face/LED display/LED matrices/U2D0D1R2
- D228 pad 2: (no net) -> /Clock face/LED display/LED matrices/U2D0D2C3
- D229 pad 1: (no net) -> /Clock face/LED display/LED matrices/U2D0D1R3
- D229 pad 2: (no net) -> /Clock face/LED display/LED matrices/U2D0D2C3
- D23 pad 1: (no net) -> Net-(D23-K)
- D23 pad 2: (no net) -> Net-(D1-A)
- D230 pad 1: (no net) -> /Clock face/LED display/LED matrices/U2D0D1R4
- D230 pad 2: (no net) -> /Clock face/LED display/LED matrices/U2D0D2C3
- D231 pad 1: (no net) -> /Clock face/LED display/LED matrices/U2D0D1R5
- D231 pad 2: (no net) -> /Clock face/LED display/LED matrices/U2D0D2C3
- D232 pad 1: (no net) -> /Clock face/LED display/LED matrices/U2D0D1R6
- D232 pad 2: (no net) -> /Clock face/LED display/LED matrices/U2D0D2C3
- D233 pad 1: (no net) -> /Clock face/LED display/LED matrices/U2D0D1R7
- D233 pad 2: (no net) -> /Clock face/LED display/LED matrices/U2D0D2C3
- D234 pad 1: (no net) -> /Clock face/LED display/LED matrices/U2D0D1R1
- D234 pad 2: (no net) -> /Clock face/LED display/LED matrices/U2D0D2C4
- D235 pad 1: (no net) -> /Clock face/LED display/LED matrices/U2D0D1R2
- D235 pad 2: (no net) -> /Clock face/LED display/LED matrices/U2D0D2C4
- D236 pad 1: (no net) -> /Clock face/LED display/LED matrices/U2D0D1R3
- D236 pad 2: (no net) -> /Clock face/LED display/LED matrices/U2D0D2C4
- D237 pad 1: (no net) -> /Clock face/LED display/LED matrices/U2D0D1R4
- D237 pad 2: (no net) -> /Clock face/LED display/LED matrices/U2D0D2C4
- D238 pad 1: (no net) -> /Clock face/LED display/LED matrices/U2D0D1R5
- D238 pad 2: (no net) -> /Clock face/LED display/LED matrices/U2D0D2C4
- D239 pad 1: (no net) -> /Clock face/LED display/LED matrices/U2D0D1R6
- D239 pad 2: (no net) -> /Clock face/LED display/LED matrices/U2D0D2C4
- D24 pad 1: (no net) -> Net-(D24-K)
- D24 pad 2: (no net) -> Net-(D1-A)
- D240 pad 1: (no net) -> /Clock face/LED display/LED matrices/U2D0D1R7
- D240 pad 2: (no net) -> /Clock face/LED display/LED matrices/U2D0D2C4
- D241 pad 1: (no net) -> /Clock face/LED display/LED matrices/U2D0D1R1
- D241 pad 2: (no net) -> /Clock face/LED display/LED matrices/U2D0D2C5
- D242 pad 1: (no net) -> /Clock face/LED display/LED matrices/U2D0D1R2
- D242 pad 2: (no net) -> /Clock face/LED display/LED matrices/U2D0D2C5
- D243 pad 1: (no net) -> /Clock face/LED display/LED matrices/U2D0D1R3
- D243 pad 2: (no net) -> /Clock face/LED display/LED matrices/U2D0D2C5
- D244 pad 1: (no net) -> /Clock face/LED display/LED matrices/U2D0D1R4
- D244 pad 2: (no net) -> /Clock face/LED display/LED matrices/U2D0D2C5
- D245 pad 1: (no net) -> /Clock face/LED display/LED matrices/U2D0D1R5
- D245 pad 2: (no net) -> /Clock face/LED display/LED matrices/U2D0D2C5
- D246 pad 1: (no net) -> /Clock face/LED display/LED matrices/U2D0D1R6
- D246 pad 2: (no net) -> /Clock face/LED display/LED matrices/U2D0D2C5
- D247 pad 1: (no net) -> /Clock face/LED display/LED matrices/U2D0D1R7
- D247 pad 2: (no net) -> /Clock face/LED display/LED matrices/U2D0D2C5
- D248 pad 1: (no net) -> /Clock face/LED display/LED matrices/U2D0D1R1
- D248 pad 2: (no net) -> /Clock face/LED display/LED matrices/U2D1D3C1
- D249 pad 1: (no net) -> /Clock face/LED display/LED matrices/U2D0D1R2
- D249 pad 2: (no net) -> /Clock face/LED display/LED matrices/U2D1D3C1
- D25 pad 1: (no net) -> Net-(D25-K)
- D25 pad 2: (no net) -> Net-(D1-A)
- D250 pad 1: (no net) -> /Clock face/LED display/LED matrices/U2D0D1R3
- D250 pad 2: (no net) -> /Clock face/LED display/LED matrices/U2D1D3C1
- D251 pad 1: (no net) -> /Clock face/LED display/LED matrices/U2D0D1R4
- D251 pad 2: (no net) -> /Clock face/LED display/LED matrices/U2D1D3C1
- D252 pad 1: (no net) -> /Clock face/LED display/LED matrices/U2D0D1R5
- D252 pad 2: (no net) -> /Clock face/LED display/LED matrices/U2D1D3C1
- D253 pad 1: (no net) -> /Clock face/LED display/LED matrices/U2D0D1R6
- D253 pad 2: (no net) -> /Clock face/LED display/LED matrices/U2D1D3C1
- D254 pad 1: (no net) -> /Clock face/LED display/LED matrices/U2D0D1R7
- D254 pad 2: (no net) -> /Clock face/LED display/LED matrices/U2D1D3C1
- D255 pad 1: (no net) -> /Clock face/LED display/LED matrices/U2D0D1R1
- D255 pad 2: (no net) -> /Clock face/LED display/LED matrices/U2D1D3C2
- D256 pad 1: (no net) -> /Clock face/LED display/LED matrices/U2D0D1R2
- D256 pad 2: (no net) -> /Clock face/LED display/LED matrices/U2D1D3C2
- D257 pad 1: (no net) -> /Clock face/LED display/LED matrices/U2D0D1R3
- D257 pad 2: (no net) -> /Clock face/LED display/LED matrices/U2D1D3C2
- D258 pad 1: (no net) -> /Clock face/LED display/LED matrices/U2D0D1R4
- D258 pad 2: (no net) -> /Clock face/LED display/LED matrices/U2D1D3C2
- D259 pad 1: (no net) -> /Clock face/LED display/LED matrices/U2D0D1R5
- D259 pad 2: (no net) -> /Clock face/LED display/LED matrices/U2D1D3C2
- D26 pad 1: (no net) -> Net-(D26-K)
- D26 pad 2: (no net) -> Net-(D1-A)
- D260 pad 1: (no net) -> /Clock face/LED display/LED matrices/U2D0D1R6
- D260 pad 2: (no net) -> /Clock face/LED display/LED matrices/U2D1D3C2
- D261 pad 1: (no net) -> /Clock face/LED display/LED matrices/U2D0D1R7
- D261 pad 2: (no net) -> /Clock face/LED display/LED matrices/U2D1D3C2
- D262 pad 1: (no net) -> /Clock face/LED display/LED matrices/U2D0D1R1
- D262 pad 2: (no net) -> /Clock face/LED display/LED matrices/U2D1D3C3
- D263 pad 1: (no net) -> /Clock face/LED display/LED matrices/U2D0D1R2
- D263 pad 2: (no net) -> /Clock face/LED display/LED matrices/U2D1D3C3
- D264 pad 1: (no net) -> /Clock face/LED display/LED matrices/U2D0D1R3
- D264 pad 2: (no net) -> /Clock face/LED display/LED matrices/U2D1D3C3
- D265 pad 1: (no net) -> /Clock face/LED display/LED matrices/U2D0D1R4
- D265 pad 2: (no net) -> /Clock face/LED display/LED matrices/U2D1D3C3
- D266 pad 1: (no net) -> /Clock face/LED display/LED matrices/U2D0D1R5
- D266 pad 2: (no net) -> /Clock face/LED display/LED matrices/U2D1D3C3
- D267 pad 1: (no net) -> /Clock face/LED display/LED matrices/U2D0D1R6
- D267 pad 2: (no net) -> /Clock face/LED display/LED matrices/U2D1D3C3
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Routing:
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- added copper zone on B.Cu, net GND
- added copper zone on In1.Cu, net GND
- added copper zone on In2.Cu, net GND
Other:
- outline, holes or cut-outs redrawn
- copper layers 2 -> 4
- board text added: "BOOT"
- board text added: "RESET"

Commit message: Routing in progress
Parts:
- U1, U2, U4: moved to B.Cu
- moved C1 10.8 mm to (57.4, 150.7)
- moved R213 10.3 mm to (237.7, 45.2)
- turned C22 to -90 degrees
- turned C23 to -90 degrees
- turned U1 to 180 degrees
- turned U2 to 180 degrees
Connections:
- net Net-(U10-VI) renamed +8.1V
- net Net-(U10-VO) renamed +5V
- C10 pad 1: Net-(U7-VCC) -> +3.3V_LED
- C11 pad 1: Net-(U8-VCC) -> +3.3V_LED
- C13 pad 1: Net-(U3-3V3) -> +3.3V_MCU
- C2 pad 1: Net-(C2-Pad1) -> +3.3V_LED
- C22 pad 1: Net-(U15-SCL) -> +3.3V_MCU
- C23 pad 1: Net-(U15-SCL) -> +3.3V_MCU
- C26 pad 1: Net-(U12-VO) -> +3.3V_GPS
- C28 pad 1: Net-(U12-VO) -> +3.3V_GPS
- C3 pad 1: Net-(C3-Pad1) -> +3.3V_LED
- C31 pad 1: Net-(U14-VO) -> +3.3V_MCU
- C32 pad 1: Net-(U13-VO) -> +3.3V_LED
- C5 pad 1: Net-(C2-Pad1) -> +3.3V_LED
- C6 pad 1: Net-(C3-Pad1) -> +3.3V_LED
- C7 pad 1: Net-(U4-VCC) -> +3.3V_LED
- C8 pad 1: Net-(U5-VCC) -> +3.3V_LED
- C9 pad 1: Net-(U6-VCC) -> +3.3V_LED
- D1 pad 2: Net-(D1-A) -> +3.3V_LED
- D10 pad 2: Net-(D1-A) -> +3.3V_LED
- D11 pad 2: Net-(D1-A) -> +3.3V_LED
- D12 pad 2: Net-(D1-A) -> +3.3V_LED
- D13 pad 2: Net-(D1-A) -> +3.3V_LED
- D14 pad 2: Net-(D1-A) -> +3.3V_LED
- D15 pad 2: Net-(D1-A) -> +3.3V_LED
- D16 pad 2: Net-(D1-A) -> +3.3V_LED
- D17 pad 2: Net-(D1-A) -> +3.3V_LED
- D18 pad 2: Net-(D1-A) -> +3.3V_LED
- D19 pad 2: Net-(D1-A) -> +3.3V_LED
- D2 pad 2: Net-(D1-A) -> +3.3V_LED
- D20 pad 2: Net-(D1-A) -> +3.3V_LED
- D21 pad 2: Net-(D1-A) -> +3.3V_LED
- D22 pad 2: Net-(D1-A) -> +3.3V_LED
- D23 pad 2: Net-(D1-A) -> +3.3V_LED
- D24 pad 2: Net-(D1-A) -> +3.3V_LED
- D25 pad 2: Net-(D1-A) -> +3.3V_LED
- D26 pad 2: Net-(D1-A) -> +3.3V_LED
- D27 pad 2: Net-(D1-A) -> +3.3V_LED
- D28 pad 2: Net-(D1-A) -> +3.3V_LED
- D29 pad 2: Net-(D1-A) -> +3.3V_LED
- D3 pad 2: Net-(D1-A) -> +3.3V_LED
- D30 pad 2: Net-(D1-A) -> +3.3V_LED
- D31 pad 2: Net-(D1-A) -> +3.3V_LED
- D32 pad 2: Net-(D1-A) -> +3.3V_LED
- D33 pad 2: Net-(D1-A) -> +3.3V_LED
- D34 pad 2: Net-(D1-A) -> +3.3V_LED
- D35 pad 2: Net-(D1-A) -> +3.3V_LED
- D353 pad 2: Net-(D353-A) -> +3.3V_LED
- D354 pad 2: Net-(D353-A) -> +3.3V_LED
- D357 pad 2: Net-(D357-A) -> +3.3V_LED
- D358 pad 2: Net-(D357-A) -> +3.3V_LED
- D359 pad 2: Net-(D357-A) -> +3.3V_LED
- D36 pad 2: Net-(D1-A) -> +3.3V_LED
- D360 pad 2: Net-(D357-A) -> +3.3V_LED
- D37 pad 2: Net-(D1-A) -> +3.3V_LED
- D38 pad 2: Net-(D1-A) -> +3.3V_LED
- D39 pad 2: Net-(D1-A) -> +3.3V_LED
- D4 pad 2: Net-(D1-A) -> +3.3V_LED
- D40 pad 2: Net-(D1-A) -> +3.3V_LED
- D41 pad 2: Net-(D1-A) -> +3.3V_LED
- D42 pad 2: Net-(D1-A) -> +3.3V_LED
- D43 pad 2: Net-(D1-A) -> +3.3V_LED
- D44 pad 2: Net-(D1-A) -> +3.3V_LED
- D45 pad 2: Net-(D1-A) -> +3.3V_LED
- D46 pad 2: Net-(D1-A) -> +3.3V_LED
- D47 pad 2: Net-(D1-A) -> +3.3V_LED
- D48 pad 2: Net-(D1-A) -> +3.3V_LED
- D49 pad 2: Net-(D1-A) -> +3.3V_LED
- D5 pad 2: Net-(D1-A) -> +3.3V_LED
- D50 pad 2: Net-(D1-A) -> +3.3V_LED
- D51 pad 2: Net-(D1-A) -> +3.3V_LED
- D52 pad 2: Net-(D1-A) -> +3.3V_LED
- D53 pad 2: Net-(D1-A) -> +3.3V_LED
- D54 pad 2: Net-(D1-A) -> +3.3V_LED
- D55 pad 2: Net-(D1-A) -> +3.3V_LED
- D56 pad 2: Net-(D1-A) -> +3.3V_LED
- D57 pad 2: Net-(D1-A) -> +3.3V_LED
- D58 pad 2: Net-(D1-A) -> +3.3V_LED
- D59 pad 2: Net-(D1-A) -> +3.3V_LED
- D6 pad 2: Net-(D1-A) -> +3.3V_LED
- D60 pad 2: Net-(D1-A) -> +3.3V_LED
- D61 pad 2: Net-(D61-A) -> +3.3V_LED
- D62 pad 2: Net-(D61-A) -> +3.3V_LED
- D63 pad 2: Net-(D61-A) -> +3.3V_LED
- D64 pad 2: Net-(D61-A) -> +3.3V_LED
- D65 pad 2: Net-(D61-A) -> +3.3V_LED
- D66 pad 2: Net-(D61-A) -> +3.3V_LED
- D67 pad 2: Net-(D61-A) -> +3.3V_LED
- D68 pad 2: Net-(D61-A) -> +3.3V_LED
- D69 pad 2: Net-(D61-A) -> +3.3V_LED
- D7 pad 2: Net-(D1-A) -> +3.3V_LED
- D70 pad 2: Net-(D61-A) -> +3.3V_LED
- D71 pad 2: Net-(D61-A) -> +3.3V_LED
- D72 pad 2: Net-(D61-A) -> +3.3V_LED
- D8 pad 2: Net-(D1-A) -> +3.3V_LED
- D9 pad 2: Net-(D1-A) -> +3.3V_LED
- J1 pad 1: Net-(J1-Pin_1) -> +3.3V_MCU
- J3 pad 1: Net-(J3-Pin_1) -> +3.3V_GPS
- R11 pad 1: Net-(R11-Pad1) -> +3.3V_LED
- R12 pad 1: Net-(R12-Pad1) -> +3.3V_MCU
- R13 pad 1: Net-(U3-3V3) -> +3.3V_MCU
- R15 pad 2: Net-(R15-Pad2) -> +3.3V_MCU
- R17 pad 1: Net-(R17-Pad1) -> +3.3V_MCU
- R18 pad 1: Net-(R18-Pad1) -> +3.3V_MCU
- R19 pad 1: Net-(R12-Pad1) -> +3.3V_MCU
- R2 pad 1: Net-(U3-3V3) -> +3.3V_MCU
- R213 pad 1: Net-(R11-Pad1) -> +3.3V_LED
- R3 pad 1: Net-(R3-Pad1) -> +3.3V_LED
- R4 pad 1: Net-(R4-Pad1) -> +3.3V_LED
- U1 pad 32: Net-(C2-Pad1) -> +3.3V_LED
- U1 pad 33: Net-(C2-Pad1) -> +3.3V_LED
- U12 pad 2: Net-(U12-VO) -> +3.3V_GPS
- U13 pad 2: Net-(U13-VO) -> +3.3V_LED
- U14 pad 2: Net-(U14-VO) -> +3.3V_MCU
- U15 pad 2: Net-(U15-SCL) -> +3.3V_MCU
- U2 pad 32: Net-(C3-Pad1) -> +3.3V_LED
- U2 pad 33: Net-(C3-Pad1) -> +3.3V_LED
- U3 pad 2: Net-(U3-3V3) -> +3.3V_MCU
- U4 pad 28: Net-(U4-VCC) -> +3.3V_LED
- U5 pad 28: Net-(U5-VCC) -> +3.3V_LED
- U6 pad 28: Net-(U6-VCC) -> +3.3V_LED
- U7 pad 28: Net-(U7-VCC) -> +3.3V_LED
- U8 pad 28: Net-(U8-VCC) -> +3.3V_LED
- U9 pad 6: Net-(J3-Pin_1) -> +3.3V_GPS
Routing:
- net +3.3V_LED: track 0.00 -> 1256.0 mm, vias 0 -> 16
- net GND: track 504.1 -> 1045.9 mm, vias 357 -> 366
- net /Clock face/LED display/LED matrices/U2D0D2C1: track 0.00 -> 329.4 mm, vias 0 -> 1
- net /Clock face/LED display/LED matrices/U2D0D2C2: track 0.00 -> 321.6 mm, vias 0 -> 1
- net /Clock face/LED display/LED matrices/U2D0D2C3: track 0.00 -> 313.7 mm, vias 0 -> 1
- net /Clock face/LED display/LED matrices/U2D0D2C4: track 0.00 -> 305.9 mm, vias 0 -> 1
- net /Clock face/LED display/LED matrices/U2D0D2C5: track 0.00 -> 298.0 mm, vias 0 -> 1
- net /Clock face/DISP_U1BLINK: track 0.00 -> 287.3 mm, vias 0 -> 2
- net /Clock face/LED display/LED matrices/U2D1D3C1: track 0.00 -> 286.1 mm, vias 0 -> 1
- net /Clock face/LED display/LED matrices/U1D1D3C5: track 0.00 -> 284.7 mm, vias 0 -> 1
- net /Clock face/LED display/LED matrices/U2D1D3C2: track 0.00 -> 278.3 mm, vias 0 -> 1
- net /Clock face/LED display/LED matrices/U1D1D3C4: track 0.00 -> 276.7 mm, vias 0 -> 1
- net /Clock face/LED display/LED matrices/U2D1D3C3: track 0.00 -> 270.7 mm, vias 0 -> 1
- net /Clock face/LED display/LED matrices/U1D1D3C3: track 0.00 -> 267.9 mm, vias 0 -> 1
- net /Clock face/LED display/LED matrices/U2D1D3C4: track 0.00 -> 262.9 mm, vias 0 -> 1
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