File: hardware/led_dial.kicad_sch (KiCad schematic)
At the start: 95 parts, among them U4 TLC5940PWP, U5 TLC5940PWP, U6 TLC5940PWP, U7 TLC5940PWP, U8 TLC5940PWP

Commit message: Assign footprints
Parts:
- C10, C11, C7, C8, C9: footprint (none) -> Capacitor_SMD:C_0805_2012Metric
- R10, R11, R213, R6, R7, R8, R9: footprint (none) -> Resistor_SMD:R_0805_2012Metric
Changed lines of the file:
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@@
       (effects (font (size 0.762 0.762)) (justify left))
     )
-    (property "Footprint" "" (at 247.65 71.12 0)
+    (property "Footprint" "Capacitor_SMD:C_0805_2012Metric" (at 247.65 71.12 0)
       (effects (font (size 1.27 1.27)) hide)
     )
@@
       (effects (font (size 0.762 0.762)) (justify left))
     )
-    (property "Footprint" "" (at 125.73 71.12 0)
+    (property "Footprint" "Capacitor_SMD:C_0805_2012Metric" (at 125.73 71.12 0)
       (effects (font (size 1.27 1.27)) hide)
     )
@@
       (effects (font (size 1.27 1.27)) (justify right))
     )
-    (property "Footprint" "" (at 198.628 73.66 90)
+    (property "Footprint" "Resistor_SMD:R_0805_2012Metric" (at 198.628 73.66 90)
       (effects (font (size 1.27 1.27)) hide)
     )
@@
       (effects (font (size 0.762 0.762)) (justify left))
     )
-    (property "Footprint" "" (at 114.3 165.1 0)
+    (property "Footprint" "Capacitor_SMD:C_0805_2012Metric" (at 114.3 165.1 0)
       (effects (font (size 1.27 1.27)) hide)
     )
@@
       (effects (font (size 0.762 0.762)) (justify left))
     )
-    (property "Footprint" "" (at 64.77 71.12 0)
+    (property "Footprint" "Capacitor_SMD:C_0805_2012Metric" (at 64.77 71.12 0)
       (effects (font (size 1.27 1.27)) hide)
     )
@@
       (effects (font (size 1.27 1.27)) (justify right))
     )
-    (property "Footprint" "" (at 76.708 73.66 90)
+    (property "Footprint" "Resistor_SMD:R_0805_2012Metric" (at 76.708 73.66 90)
       (effects (font (size 1.27 1.27)) hide)
     )
@@
       (effects (font (size 1.27 1.27)) (justify right))
     )
-    (property "Footprint" "" (at 102.362 167.64 90)
+    (property "Footprint" "Resistor_SMD:R_0805_2012Metric" (at 102.362 167.64 90)
       (effects (font (size 1.27 1.27)) hide)
     )
@@
       (effects (font (size 0.762 0.762)) (justify left))
     )
-    (property "Footprint" "" (at 186.69 71.12 0)
+    (property "Footprint" "Capacitor_SMD:C_0805_2012Metric" (at 186.69 71.12 0)
       (effects (font (size 1.27 1.27)) hide)
     )
@@
       (effects (font (size 1.27 1.27)) (justify right))
     )
-    (property "Footprint" "" (at 48.768 119.38 90)
+    (property "Footprint" "Resistor_SMD:R_0805_2012Metric" (at 48.768 119.38 90)
       (effects (font (size 1.27 1.27)) hide)
     )
@@
       (effects (font (size 1.27 1.27)) (justify right))
     )
-    (property "Footprint" "" (at 38.608 119.38 90)
+    (property "Footprint" "Resistor_SMD:R_0805_2012Metric" (at 38.608 119.38 90)
       (effects (font (size 1.27 1.27)) hide)
     )
@@
       (effects (font (size 1.27 1.27)) (justify right))
     )
-    (property "Footprint" "" (at 137.668 73.66 90)
+    (property "Footprint" "Resistor_SMD:R_0805_2012Metric" (at 137.668 73.66 90)
       (effects (font (size 1.27 1.27)) hide)
     )
@@
       (effects (font (size 1.27 1.27)) (justify right))
     )
-    (property "Footprint" "" (at 259.588 73.66 90)
-      (effects (font (size 1.27 1.27)) hide)
-    )
+    (property "Footprint" "Resistor_SMD:R_0805_2012Metric" (at 259.588 73.66 90)
+      (effects (font (size 1.27 1.27)) hide)
+    )

Commit message: Starting PCB routing process
Parts:
- R11: value 100k -> R
- U4, U5, U6, U7, U8: footprint Package_SO:HTSSOP-28-1EP_4.4x9.7mm_P0.65mm_EP3.4x9.5mm_Mask2.4x6.17mm_ThermalVias -> Package_SO_espena:HTSSOP-28-1EP_4.4x9.7mm_P0.65mm_EP3.4x9.5mm_Mask2.4x6.17mm_ThermalVias
Connections:
- net at R213.1: now also R11.1

Commit message: Routing in progress
Connections:
- net +3.3V_LED: now reaches D1.2 (A), D10.2 (A), D11.2 (A), D12.2 (A), D13.2 (A), D14.2 (A), D15.2 (A), D16.2 (A), D17.2 (A), D18.2 (A), D19.2 (A), D2.2 (A), D20.2 (A), D21.2 (A), D22.2 (A), D23.2 (A), D24.2 (A), D25.2 (A), D26.2 (A), D27.2 (A), D28.2 (A), D29.2 (A), D3.2 (A), D30.2 (A), D31.2 (A), D32.2 (A), D33.2 (A), D34.2 (A), D35.2 (A), D36.2 (A), D37.2 (A), D38.2 (A), D39.2 (A), D4.2 (A), D40.2 (A), D41.2 (A), D42.2 (A), D43.2 (A), D44.2 (A), D45.2 (A), D46.2 (A), D47.2 (A), D48.2 (A), D49.2 (A), D5.2 (A), D50.2 (A), D51.2 (A), D52.2 (A), D53.2 (A), D54.2 (A), D55.2 (A), D56.2 (A), D57.2 (A), D58.2 (A), D59.2 (A), D6.2 (A), D60.2 (A), D7.2 (A), D8.2 (A), D9.2 (A)
- net +3.3V_LED: now also C10.1, C11.1, C7.1, C8.1, C9.1, D353.2 (A), D354.2 (A), D357.2 (A), D358.2 (A), D359.2 (A), D360.2 (A), D61.2 (A), D62.2 (A), D63.2 (A), D64.2 (A), D65.2 (A), D66.2 (A), D67.2 (A), D68.2 (A), D69.2 (A), D70.2 (A), D71.2 (A), D72.2 (A), R11.1, R213.1, U4.28 (VCC), U5.28 (VCC), U6.28 (VCC), U7.28 (VCC), U8.28 (VCC)
Changed lines of the file:
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@@
 		(on_board yes)
 		(dnp no)
-		(property "Reference" "#PWR018"
+		(property "Reference" "#PWR_LED018"
 			(at 238.76 82.55 0)
 			(effects
@@
 			)
 		)
-		(property "Description" "Power symbol creates a global label with name \"+3.3V\""
+		(property "Description" "Power symbol creates a global label with name \"PWR_LED\""
 			(at 238.76 78.74 0)
 			(effects
@@
 			(project "broadcast_clock"
 				(path "/40ecfd14-7e3d-4342-87f4-c464dfcd4cdf/425f15d8-7995-473a-916f-1acbbdb328a4/a3edaa85-e896-4c15-8162-60d9cf8f1ed2"
-					(reference "#PWR018")
+					(reference "#PWR_LED018")
 					(unit 1)
 				)
@@
 		(on_board yes)
 		(dnp no)
-		(property "Reference" "#PWR012"
+		(property "Reference" "#PWR_LED012"
 			(at 116.84 82.55 0)
 			(effects
@@
 			)
 		)
-		(property "Description" "Power symbol creates a global label with name \"+3.3V\""
+		(property "Description" "Power symbol creates a global label with name \"PWR_LED\""
 			(at 116.84 78.74 0)
 			(effects
@@
 			(project "broadcast_clock"
 				(path "/40ecfd14-7e3d-4342-87f4-c464dfcd4cdf/425f15d8-7995-473a-916f-1acbbdb328a4/a3edaa85-e896-4c15-8162-60d9cf8f1ed2"
-					(reference "#PWR012")
+					(reference "#PWR_LED012")
 					(unit 1)
 				)
@@
 		(on_board yes)
 		(dnp no)
-		(property "Reference" "#PWR015"
+		(property "Reference" "#PWR_LED015"
 			(at 177.8 82.55 0)
 			(effects
@@
 			)
 		)
-		(property "Description" "Power symbol creates a global label with name \"+3.3V\""
+		(property "Description" "Power symbol creates a global label with name \"PWR_LED\""
 			(at 177.8 78.74 0)
 			(effects
@@
 			(project "broadcast_clock"
 				(path "/40ecfd14-7e3d-4342-87f4-c464dfcd4cdf/425f15d8-7995-473a-916f-1acbbdb328a4/a3edaa85-e896-4c15-8162-60d9cf8f1ed2"
-					(reference "#PWR015")
+					(reference "#PWR_LED015")
 					(unit 1)
 				)
@@
 		(on_board yes)
 		(dnp no)
-		(property "Reference" "#PWR08"
+		(property "Reference" "#PWR_LED08"
 			(at 148.59 120.65 0)
 			(effects
@@
 			)
 		)
-		(property "Description" "Power symbol creates a global label with name \"+3.3V\""
+		(property "Description" "Power symbol creates a global label with name \"PWR_LED\""
 			(at 148.59 116.84 0)
 			(effects
@@
 			(project "broadcast_clock"
 				(path "/40ecfd14-7e3d-4342-87f4-c464dfcd4cdf/425f15d8-7995-473a-916f-1acbbdb328a4/a3edaa85-e896-4c15-8162-60d9cf8f1ed2"
-					(reference "#PWR08")
+					(reference "#PWR_LED08")
 					(unit 1)
 				)
@@
 		(on_board yes)
 		(dnp no)
-		(property "Reference" "#PWR0223"
+		(property "Reference" "#PWR_LED0223"
 			(at 46.99 116.84 0)
 			(effects
@@
 			)
 		)
-		(property "Description" "Power symbol creates a global label with name \"+3.3V\""
+		(property "Description" "Power symbol creates a global label with name \"PWR_LED\""
 			(at 46.99 113.03 0)
 			(effects
@@
 			(project "broadcast_clock"
 				(path "/40ecfd14-7e3d-4342-87f4-c464dfcd4cdf/425f15d8-7995-473a-916f-1acbbdb328a4/a3edaa85-e896-4c15-8162-60d9cf8f1ed2"
-					(reference "#PWR0223")
+					(reference "#PWR_LED0223")
 					(unit 1)
 				)
@@
 		(on_board yes)
 		(dnp no)
-		(property "Reference" "#PWR065"
+		(property "Reference" "#PWR_LED065"
 			(at 259.08 26.035 0)
 			(effects
@@
 			)
 		)
-		(property "Description" "Power symbol creates a global label with name \"+3.3V\""
+		(property "Description" "Power symbol creates a global label with name \"PWR_LED\""
 			(at 259.08 22.225 0)
 			(effects
@@
 			(project "broadcast_clock"
 				(path "/40ecfd14-7e3d-4342-87f4-c464dfcd4cdf/425f15d8-7995-473a-916f-1acbbdb328a4/a3edaa85-e896-4c15-8162-60d9cf8f1ed2"
-					(reference "#PWR065")
+					(reference "#PWR_LED065")
 					(unit 1)
 				)
@@
 		(on_board yes)
 		(dnp no)
-		(property "Reference" "#PWR0224"
+		(property "Reference" "#PWR_LED0224"
 			(at 95.25 120.65 0)
 			(effects
@@
 			)
 		)
-		(property "Description" "Power symbol creates a global label with name \"+3.3V\""
+		(property "Description" "Power symbol creates a global label with name \"PWR_LED\""
 			(at 95.25 116.84 0)
 			(effects
@@
 			(project "broadcast_clock"
 				(path "/40ecfd14-7e3d-4342-87f4-c464dfcd4cdf/425f15d8-7995-473a-916f-1acbbdb328a4/a3edaa85-e896-4c15-8162-60d9cf8f1ed2"
-					(reference "#PWR0224")
+					(reference "#PWR_LED0224")
 					(unit 1)
 				)
@@
 		(on_board yes)
 		(dnp no)
-		(property "Reference" "#PWR07"
+		(property "Reference" "#PWR_LED07"
 			(at 30.48 26.035 0)
 			(effects
@@
 			)
 		)
-		(property "Description" "Power symbol creates a global label with name \"+3.3V\""
+		(property "Description" "Power symbol creates a global label with name \"PWR_LED\""
 			(at 30.48 22.225 0)
 			(effects
@@
 			(project "broadcast_clock"
 				(path "/40ecfd14-7e3d-4342-87f4-c464dfcd4cdf/425f15d8-7995-473a-916f-1acbbdb328a4/a3edaa85-e896-4c15-8162-60d9cf8f1ed2"
-					(reference "#PWR07")
+					(reference "#PWR_LED07")
 					(unit 1)
 				)
@@
 		(on_board yes)
 		(dnp no)
-		(property "Reference" "#PWR021"
+		(property "Reference" "#PWR_LED021"
 			(at 123.19 176.53 0)
 			(effects
@@
 			)
 		)
-		(property "Description" "Power symbol creates a global label with name \"+3.3V\""
+		(property "Description" "Power symbol creates a global label with name \"PWR_LED\""
 			(at 123.19 172.72 0)
 			(effects
@@
 			(project "broadcast_clock"
 				(path "/40ecfd14-7e3d-4342-87f4-c464dfcd4cdf/425f15d8-7995-473a-916f-1acbbdb328a4/a3edaa85-e896-4c15-8162-60d9cf8f1ed2"
-					(reference "#PWR021")
+					(reference "#PWR_LED021")
 					(unit 1)
 				)
@@
 		(on_board yes)
 		(dnp no)
-		(property "Reference" "#PWR09"
+		(property "Reference" "#PWR_LED09"
 			(at 55.88 82.55 0)
 			(effects
@@
 			)
 		)
-		(property "Description" "Power symbol creates a global label with name \"+3.3V\""
+		(property "Description" "Power symbol creates a global label with name \"PWR_LED\""
 			(at 55.88 78.74 0)
 			(effects
@@
 			(project "broadcast_clock"
 				(path "/40ecfd14-7e3d-4342-87f4-c464dfcd4cdf/425f15d8-7995-473a-916f-1acbbdb328a4/a3edaa85-e896-4c15-8162-60d9cf8f1ed2"
-					(reference "#PWR09")
+					(reference "#PWR_LED09")
 					(unit 1)
 				)

Commit message: Open thermal pad for buck converter
Former-commit-id: e6c8dc76280dd95d3ab8586baa877e8ee88db5e2
Parts:
- U4, U5, U6, U7, U8: footprint Package_SO_espena:HTSSOP-28-1EP_4.4x9.7mm_P0.65mm_EP3.4x9.5mm_Mask2.4x6.17mm_ThermalVias -> Package_SO:HTSSOP-28-1EP_4.4x9.7mm_P0.65mm_EP3.4x9.5mm_Mask2.4x6.17mm_ThermalVias
Changed lines of the file:
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@@
 			)
 		)
-		(property "Footprint" "Package_SO_espena:HTSSOP-28-1EP_4.4x9.7mm_P0.65mm_EP3.4x9.5mm_Mask2.4x6.17mm_ThermalVias"
+		(property "Footprint" "Package_SO:HTSSOP-28-1EP_4.4x9.7mm_P0.65mm_EP3.4x9.5mm_Mask2.4x6.17mm_ThermalVias"
 			(at 192.405 50.165 0)
 			(effects
@@
 			)
 		)
-		(property "Footprint" "Package_SO_espena:HTSSOP-28-1EP_4.4x9.7mm_P0.65mm_EP3.4x9.5mm_Mask2.4x6.17mm_ThermalVias"
+		(property "Footprint" "Package_SO:HTSSOP-28-1EP_4.4x9.7mm_P0.65mm_EP3.4x9.5mm_Mask2.4x6.17mm_ThermalVias"
 			(at 253.365 50.165 0)
 			(effects
@@
 			)
 		)
-		(property "Footprint" "Package_SO_espena:HTSSOP-28-1EP_4.4x9.7mm_P0.65mm_EP3.4x9.5mm_Mask2.4x6.17mm_ThermalVias"
+		(property "Footprint" "Package_SO:HTSSOP-28-1EP_4.4x9.7mm_P0.65mm_EP3.4x9.5mm_Mask2.4x6.17mm_ThermalVias"
 			(at 70.485 50.165 0)
 			(effects
@@
 			)
 		)
-		(property "Footprint" "Package_SO_espena:HTSSOP-28-1EP_4.4x9.7mm_P0.65mm_EP3.4x9.5mm_Mask2.4x6.17mm_ThermalVias"
+		(property "Footprint" "Package_SO:HTSSOP-28-1EP_4.4x9.7mm_P0.65mm_EP3.4x9.5mm_Mask2.4x6.17mm_ThermalVias"
 			(at 131.445 50.165 0)
 			(effects
@@
 			)
 		)
-		(property "Footprint" "Package_SO_espena:HTSSOP-28-1EP_4.4x9.7mm_P0.65mm_EP3.4x9.5mm_Mask2.4x6.17mm_ThermalVias"
+		(property "Footprint" "Package_SO:HTSSOP-28-1EP_4.4x9.7mm_P0.65mm_EP3.4x9.5mm_Mask2.4x6.17mm_ThermalVias"
 			(at 108.585 144.145 0)
 			(effects

Commit message: Prototype, starting on firmware
Former-commit-id: 3c22e4f94bda4a4eed472ac1ff762e7709731c05
Former-commit-id: afce4fecf5b4961621dea2f3a514203675ae8e80
Parts:
- R11: value R -> 10k
Changed lines of the file:
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@@
 			)
 		)
-		(property "Value" "R"
+		(property "Value" "10k"
 			(at 41.275 120.6499 0)
 			(effects

Commit message: Minor design updates
Parts:
- R10, R6, R7, R8, R9: value 2k -> 2kΩ
- R11, R213: value 10k -> 10kΩ
Changed lines of the file:
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@@
 		(fields_autoplaced yes)
 		(property "Reference" "R8"
-			(at 199.39 73.025 0)
+			(at 199.39 72.3899 0)
 			(effects
 				(font
@@
 			)
 		)
-		(property "Value" "2k"
-			(at 199.39 75.565 0)
+		(property "Value" "2kΩ"
+			(at 199.39 74.9299 0)
 			(effects
 				(font
@@
 		(fields_autoplaced yes)
 		(property "Reference" "R6"
-			(at 77.47 73.025 0)
+			(at 77.47 72.3899 0)
 			(effects
 				(font
@@
 			)
 		)
-		(property "Value" "2k"
-			(at 77.47 75.565 0)
+		(property "Value" "2kΩ"
+			(at 77.47 74.9299 0)
 			(effects
 				(font
@@
 		(fields_autoplaced yes)
 		(property "Reference" "R10"
-			(at 101.6 167.005 0)
+			(at 106.68 166.3699 0)
 			(effects
 				(font
 					(size 1.27 1.27)
 				)
-				(justify right)
+				(justify left)
 			)
 		)
-		(property "Value" "2k"
-			(at 101.6 169.545 0)
+		(property "Value" "2kΩ"
+			(at 106.68 168.9099 0)
 			(effects
 				(font
 					(size 1.27 1.27)
 				)
-				(justify right)
+				(justify left)
 			)
 		)
@@
 		(fields_autoplaced yes)
 		(property "Reference" "R213"
-			(at 49.53 118.745 0)
+			(at 49.53 118.1099 0)
 			(effects
 				(font
@@
 			)
 		)
-		(property "Value" "10k"
-			(at 49.53 121.285 0)
+		(property "Value" "10kΩ"
+			(at 49.53 120.6499 0)
 			(effects
 				(font
@@
 		(fields_autoplaced yes)
 		(property "Reference" "R7"
-			(at 138.43 73.025 0)
+			(at 138.43 72.3899 0)
 			(effects
 				(font
@@
 			)
 		)
-		(property "Value" "2k"
-			(at 138.43 75.565 0)
+		(property "Value" "2kΩ"
+			(at 138.43 74.9299 0)
 			(effects
 				(font
@@
 		(fields_autoplaced yes)
 		(property "Reference" "R9"
-			(at 260.35 73.025 0)
+			(at 260.35 72.3899 0)
 			(effects
 				(font
@@
 			)
 		)
-		(property "Value" "2k"
-			(at 260.35 75.565 0)
+		(property "Value" "2kΩ"
+			(at 260.35 74.9299 0)
 			(effects
 				(font
@@
 			)
 		)
-		(property "Value" "10k"
+		(property "Value" "10kΩ"
 			(at 41.275 120.6499 0)
 			(effects
